Commit message: feat: gazebo simulation integrated in oculus

File: urdf/hmd_head.urdf (robot description, URDF)
Before this commit: robot hmd_head, 7 links, 6 joints
Links:
- removed link indicator_x
- removed link indicator_y
- removed link indicator_z
- added link camera_link, mass 0.02; collision box size=0.02 0.04 0.04; visual box size=0.02 0.04 0.04
- added link camera_optical_frame
Joints:
- removed joint head_to_indicator
- removed joint head_to_indicator_y
- removed joint head_to_indicator_z
- added joint camera_optical_joint: type fixed, parent camera_link, child camera_optical_frame, origin xyz=0 0 0 rpy=-1.57079632679 0 -1.57079632679
- added joint head_to_camera: type fixed, parent head_link, child camera_link, origin xyz=0.09 0 0 rpy=0 0 0

Commit message: feat: new robot model

File: urdf/hmd_head.urdf (robot description, URDF)
Before this commit: robot hmd_head, 6 links, 5 joints
Links:
- added link wheel_back_sphere, mass 0.5; collision sphere radius=0.06; visual sphere radius=0.06
- added link wheel_front_left_sphere, mass 0.5; collision sphere radius=0.06; visual sphere radius=0.06
- added link wheel_front_right_sphere, mass 0.5; collision sphere radius=0.06; visual sphere radius=0.06
- link base_link: mass 0.5 -> 18.0; geometry collision box size=0.48 0.48 0.08; visual box size=0.48 0.48 0.08
- link camera_link: mass 0.02 -> 0.5; geometry collision box size=0.05 0.07 0.07; visual box size=0.05 0.07 0.07
- link head_link: mass 0.4 -> 1.0; geometry collision sphere radius=0.15; visual sphere radius=0.15
- link neck_pitch_link: mass 0.2 -> 1.5; geometry collision cylinder length=0.06 radius=0.2; visual cylinder length=0.2 radius=0.05
- link neck_yaw_link: mass 0.2 -> 6.0; geometry collision cylinder length=1.0 radius=0.15; visual cylinder length=1.0 radius=0.15
Joints:
- added joint wheel_back_joint: type fixed, parent base_link, child wheel_back_sphere, origin xyz=-0.18 0 -0.06 rpy=0 0 0
- added joint wheel_front_left_joint: type fixed, parent base_link, child wheel_front_left_sphere, origin xyz=0.18 0.18 -0.06 rpy=0 0 0
- added joint wheel_front_right_joint: type fixed, parent base_link, child wheel_front_right_sphere, origin xyz=0.18 -0.18 -0.06 rpy=0 0 0
- joint head_roll: origin xyz=0 0 0.06 rpy=0 0 0 -> xyz=0 0 0.2 rpy=0 0 0
- joint head_to_camera: origin xyz=0.09 0 0 rpy=0 0 0 -> xyz=0.15 0 0 rpy=0 0 0
- joint neck_pitch: origin xyz=0 0 0.06 rpy=0 0 0 -> xyz=0 0 0.55 rpy=0 0 0
- joint neck_yaw: limit lower=-3.1415 upper=3.1415 effort=5 velocity=6.0 -> (none); origin xyz=0 0 0.06 rpy=0 0 0 -> xyz=0 0 0.5 rpy=0 0 0; type revolute -> continuous
